File: schematics/src/mainboard/mainboard.sch (EAGLE design)
At the start: 25 parts, among them IC1 MCP4921P, IC3 TL082P, IC4 TINY24/44/84-PU, Q1 16Mhz, T1 3904

Commit message: Updated Schematics & Firmware
Parts:
- added C12, C5, C6: 10uf, resistor:CPOL-USE2.5-5
- added C13, C14, C16, C17, C18: .1uF, rcl:C-EU050-024X044
- added C15: 47pF, rcl:C-EU050-024X044
- added CV_OFFSET: 20k, pot:TRIM_1234-S64YW
- added D1, D2: 1N4148, diode:1N4148DO35-7
- added D3, D4, D5, D6: 1n4148, diode:1N4148DO35-7
- added IC2, IC5, IC7: TL084P, linear:TL084P
- added IC6: 4013N, 40xx:4013N
- added IO_CON1, IO_CON2: (no value), pinhead:PINHD-1X4
- added JP1: (no value), pinhead:PINHD-2X3
- added PWR: (no value), con-ml:ML10
- added PWR_CON: (no value), pinhead:PINHD-1X3
- added R12, R25: 47k, rcl:R-US_0207/7
- added R13: 33k, rcl:R-US_0207/7
- added R14: 27k, rcl:R-US_0207/7
- added R15, R16, R17, R21, R30, R34: 100k .1%, rcl:R-US_0207/7
- added R18, R31: 200k .1%, rcl:R-US_0207/7
- added R19, R26: 6.8k, rcl:R-US_0207/7
- added R20: 68k, rcl:R-US_0207/7
- added R22, R24: 300k, rcl:R-US_0207/7
- added R23, R32, R42: 150k, rcl:R-US_0207/7
- added R27: 20k 1%, rcl:R-US_0207/7
- added R28: 24k 1%, rcl:R-US_0207/7
- added R29: 18k, rcl:R-US_0207/7
- added R33: 50k .1%, rcl:R-US_0207/7
- added R35, R38: 10k, rcl:R-US_0207/7
- added R36: 470k, rcl:R-US_0207/7
- added R37: 12k, rcl:R-US_0207/7
- added R39: 22k, rcl:R-US_0207/7
- added R40: 15k, rcl:R-US_0207/7
- added R41: 1.2k, rcl:R-US_0207/7
- added TP1, TP2: (no value), pinhead:PINHD-1X1
- added VREF_SET: 100k, pot:TRIM_1234-S64YW
- added VREF_SET1: 50k, pot:TRIM_1234-S64YW
- C2: value (none) -> 1.5nF
- IC3: value TL082P -> 7805L; device linear:TL082P -> linear:7805L
- Q1: value 16Mhz -> 20Mhz
- R1: value 200k -> 200k .1%
- R11: value 100k -> 150k; device pot:TRIM_1234-S64YW -> rcl:R-US_0207/7
- R5: value 100k -> 100k .1%
- R6: value 100k -> 33k .1%
- R7: value (none) -> 10k
Connections:
- removed net INT_SAW_OUT: C1.2, IC3A.OUT, R2.1
- removed net MOSI: IC1.SDI
- new net CV_INPUT: IO_CON1.2, R16.2
- new net INT_SAW: C1.2, IC2A.OUT, R2.1, R28.2
- new net MISO: IC1.SDI, IC4.(PCINT5/OC1B/MISO/DO/ADC5)PA5, JP1.1
- new net N$14: CV_OFFSET.A, R14.2
- new net N$15: CV_OFFSET.E, R13.1
- new net N$16: CV_OFFSET.S, IC2C.+IN, TP1.1
- new net N$17: IC2C.-IN, R15.2, R16.1
- new net N$18: IC6A.!Q, IC6A.D
- new net N$19: IC2C.OUT, R15.1, R17.2
- new net N$20: IC2D.-IN, R17.1, R18.2
- new net N$21: IC5B.-IN, R23.1, R24.2
- new net N$22: IC5A.-IN, R11.1, R22.2
- new net N$23: IC5A.+IN, R12.2, R19.1
- new net N$24: IC5B.+IN, R25.2, R26.1
- new net N$25: IC5D.+IN, R20.2, R29.1
- new net N$26: IC5D.-IN, R27.2, R28.1
- new net N$27: C15.2, IC7B.-IN, R21.2, R31.1, R32.1, R33.1
- new net N$28: D3.C, IC7A.-IN, R30.1, R34.2
- new net N$29: D3.A, D4.C, IC7A.OUT
- new net N$30: D4.A, R30.2, R33.2
- new net N$31: IC7C.OUT, R37.1
- new net N$32: IC7C.-IN, R35.2
- new net N$33: D5.A, D6.C, IC5C.+IN, R39.1, R42.2
- new net N$34: R32.2, VREF_SET1.S
- new net N$35: IC7D.-IN, IC7D.OUT
- new net N$36: IC5C.-IN, R40.1, R41.2
- new net PULSE_OUT: IO_CON2.4, R37.2, R38.2
- new net PWM_SET: IC7C.+IN, IO_CON1.1, R36.2
- new net RST: IC4.(PCINT11/RESET/DW)PB3, JP1.5, R7.2
- new net SAW_OUT: IC5D.OUT, IO_CON2.2, R21.1, R27.1, R34.1, R35.1
- new net SINE_OUT: IC5C.OUT, IO_CON2.3, R40.2
- new net SQR_OUT: IC5A.OUT, IO_CON1.4, R22.1
- new net SUB_SQR_OUT: IC5B.OUT, IO_CON1.3, R24.1
- new net TRI_OUT: C15.1, IC7B.OUT, IO_CON2.1, R31.2, R42.1
- net +12V: now also C14.2, C17.2, C5.+, IC2P.V+, IC3.VI, IC5P.V+, IC7P.V+, PWR.1, PWR.2, PWR_CON.3, R12.1, R13.2, R20.1, R25.1, VREF_SET1.E; no longer IC3P.V+
- net +5V: now also C12.+, C18.2, D2.C, IC3.VO, IC6P.VDD, JP1.2
- net -12V: now also C13.2, C16.2, C6.-, IC2P.V-, IC5P.V-, IC7P.V-, PWR.10, PWR.9, PWR_CON.1, R14.1; no longer IC3P.V-
- net CLOCK: now also IC4.(PCINT6/OC1A/SDA/MOSI/ADC6)PA6, IC6A.CLK, JP1.4, R11.2; no longer IC4.(PCINT10/INT0/OC0A/CKOUT)PB2
- net DAC_CS: now also IC4.(PCINT3/T0/ADC3)PA3
- net FRQ_SET: now also D1.C, D2.A, IC2D.OUT, R18.1
- net GND: now also C12.-, C13.1, C14.1, C16.1, C17.1, C18.1, C5.-, C6.+, D1.A, D5.C, D6.A, IC2A.+IN, IC2B.+IN, IC2D.+IN, IC3.GND, IC6A.R, IC6A.S, IC6B.R, IC6B.S, IC6P.VSS, IC7A.+IN, IC7B.+IN, IC7D.+IN, JP1.6, PWR.3, PWR.4, PWR.5, PWR.6, PWR.7, PWR.8, PWR_CON.2, R19.2, R26.2, R29.2, R36.1, R38.1, R39.2, R41.1, VREF_SET1.A; no longer IC3A.+IN, IC3B.+IN
- net N$1: now also IC2A.-IN; no longer IC3A.-IN
- net N$10: now also IC6A.Q, R23.2; no longer IC4.(PCINT11/RESET/DW)PB3, R7.2
- net N$12: now also VREF_SET.A; no longer R11.A
- net N$13: now also VREF_SET.S; no longer R11.S
- net N$4: now also VREF_SET.E; no longer R11.E
- net N$6: now also IC2B.OUT; no longer IC3B.OUT
- net N$8: now also IC2B.-IN; no longer IC3B.-IN
- net SCK: now also IC4.(PCINT4/T1/SCL/USCK/ADC4)PA4, JP1.3
- net VREF: now also TP2.1
Other:
- note added: "Adjust CV_OFFSET pot to get a offset of -1.50V @ TP1"
- note added: "Adjust VREF_SET pot to get 4.00V @ TP2"
- moved on the sheet: C1, C10, C2, C3, C4, C7, C8, C9, IC1, IC4, Q1, R1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

Commit message: Updated Schematics, Fixed Power Socket orientation
Parts:
- removed C5, C6: 10uf, resistor:CPOL-USE2.5-5
- added C11, C19: 10uf, resistor:CPOL-USE2.5-5
- C1: device rcl:C-EU050-024X044 -> rcl:C-EU050-025X075
- renumbered JP1 to ICSP, VREF_SET1 to TRI_SINE_SYM
Connections:
- net +12V: now also C19.+, PWR.10, PWR.9; no longer C5.+, PWR.1, PWR.2
- net -12V: now also C11.-, PWR.1, PWR.2; no longer C6.-, PWR.10, PWR.9
- net CV_INPUT: now also IO_CON1.4; no longer IO_CON1.2
- net GND: now also C11.+, C19.-; no longer C5.-, C6.+
- net PULSE_OUT: now also IO_CON2.3; no longer IO_CON2.4
- net SAW_OUT: now also IO_CON2.1; no longer IO_CON2.2
- net SINE_OUT: now also IO_CON2.2; no longer IO_CON2.3
- net SQR_OUT: now also IO_CON1.3; no longer IO_CON1.4
- net SUB_SQR_OUT: now also IO_CON1.2; no longer IO_CON1.3
- net TRI_OUT: now also IO_CON2.4; no longer IO_CON2.1
Other:
- moved on the sheet: IO_CON2, PWR
